Commit message: Fixed in JointStatePublisher::setPublishCycle() and implemented multi_lwr4p_robots_test

File: src/test/robot_test/urdf/multi_lwr4p_robots_test.xacro (robot description, xacro)
@@ -4,9 +4,4 @@
 <!-- Import all Gazebo-customization elements, including Gazebo colors -->
 <xacro:include filename="$(find lwr4p)/urdf/kuka_lwr_arm.gazebo"/>
-<!-- Inserts the Kuka here with a specified name and direction ... -->
-<xacro:kuka_lwr_arm parent="world" name="lwr" right="1" tool_name=""/>
-<xacro:kuka_lwr_arm_gazebo name="lwr"/>
-<xacro:kuka_lwr_arm parent="world" name="lwr" right="1" tool_name=""/>
-<xacro:kuka_lwr_arm_gazebo name="lwr"/>
 <link name="world" />
 <!--
@@ -14,5 +9,5 @@
 -->
 <joint name="world_to_base1" type="fixed">
-   <origin xyz="1 0 0" rpy="0 0 0"/>
+   <origin xyz="0.8 -0.5 0" rpy="0 0 0"/>
    <parent link="world"/>
    <child link="base1"/>
@@ -25,5 +20,5 @@
 -->
 <joint name="world_to_base2" type="fixed">
-   <origin xyz="-1 0 0" rpy="0 0 0"/>
+   <origin xyz="-0.8 0.5 0" rpy="0 0 0"/>
    <parent link="world"/>
    <child link="base2"/>
@@ -32,3 +27,14 @@
 <xacro:kuka_lwr_arm parent="base2" name="lwr2" right="1" tool_name=""/>
 <xacro:kuka_lwr_arm_gazebo name="lwr2"/>
+<!--
+======  set up 3rd robot  ======
+-->
+<joint name="world_to_base3" type="fixed">
+   <origin xyz="1.15 1.2 0" rpy="0 0 0"/>
+   <parent link="world"/>
+   <child link="base3"/>
+</joint>
+<link name="base3" />
+<xacro:kuka_lwr_arm parent="base3" name="lwr3" right="1" tool_name=""/>
+<xacro:kuka_lwr_arm_gazebo name="lwr3"/>
 </robot>
