Commit message: Tested simulation of lwr4p and bhand

File: src/test/bhand_test/urdf/multi_bh282_robots_test.xacro (robot description, xacro)
@@ -9,5 +9,5 @@
 -->
 <joint name="world_to_base1" type="fixed">
-   <origin xyz="0.4 -0.2 0" rpy="0 0 0"/>
+   <origin xyz="0.0 -0.2 0" rpy="0 0 0"/>
    <parent link="world"/>
    <child link="base1"/>
@@ -21,5 +21,5 @@
 -->
 <joint name="world_to_base2" type="fixed">
-   <origin xyz="-0.4 0.2 0" rpy="0 0 0"/>
+   <origin xyz="-0.2 0.2 0" rpy="0 0 0"/>
    <parent link="world"/>
    <child link="base2"/>
@@ -33,5 +33,5 @@
 -->
 <joint name="world_to_base3" type="fixed">
-   <origin xyz="0.3 0.2 0" rpy="0 0 0"/>
+   <origin xyz="0.2 0.15 0" rpy="0 0 0"/>
    <parent link="world"/>
    <child link="base3"/>
